File: PCB_rev0/binulator_kicad_project/file5B9A3213.sch (KiCad schematic (older format))
At the start: 4 parts

Commit message: adding bulk of the components to the power schematic
Parts:
- SW?: Supplier Mouser -> (none); Supplier 1 (none) -> Mouser; Supplier 1 Order Code (none) -> 642-AKTSC21I; Supplier 2 (none) -> Digikey; Supplier 2 Order Code (none) -> 679-2313-ND; Supplier Order Code 642-AKTSC21I -> (none)
- SW?: footprint (none) -> my_footprints:ADTS648_V; Supplier Mouser -> (none); Supplier 1 (none) -> Mouser; Supplier 1 Order Code (none) -> 642-ADTS648RV; Supplier 2 (none) -> Digikey; Supplier 2 Order Code (none) -> 679-2377-ND; Supplier Order Code 642-ADTS24NV -> (none)
- SW?: value CAP_BROWN_6mm -> CAP_GREEN_6mm; Supplier Mouser -> (none); Supplier 1 (none) -> Mouser; Supplier 1 Order Code (none) -> 642-AKTSC61G
- SW?: footprint (none) -> my_footprints:ADTS24_V; Supplier Mouser -> (none); Supplier 1 (none) -> Mouser; Supplier 1 Order Code (none) -> 642-ADTS24NV; Supplier 2 (none) -> Digikey; Supplier 2 Order Code (none) -> 679-2374-ND; Supplier Order Code 642-ADTS24NV -> (none)
Changed lines of the file:
@@
 EESchema Schematic File Version 4
+LIBS:binulator_kicad_project-cache
 EELAYER 26 0
 EELAYER END
@@
 F 2 "" H 6500 3500 50  0001 C CNN
 F 3 "~" H 6500 3500 50  0001 C CNN
-F 4 "Mouser" H 6500 3500 50  0001 C CNN "Supplier"
-F 5 "642-AKTSC21I " H 6500 3500 50  0001 C CNN "Supplier Order Code"
+F 4 "Mouser" H 6500 3500 50  0001 C CNN "Supplier 1"
+F 5 "642-AKTSC21I" H 6500 3500 50  0001 C CNN "Supplier 1 Order Code"
+F 6 "Digikey" H 6500 3500 50  0001 C CNN "Supplier 2"
+F 7 "679-2313-ND" H 6500 3500 50  0001 C CNN "Supplier 2 Order Code"
 	1    6500 3500
 	1    0    0    -1
@@
 F 0 "SW?" V 5654 3730 50  0000 L CNN
 F 1 "SW_12mm" V 5745 3730 50  0000 L CNN
-F 2 "" H 5700 3500 50  0001 C CNN
+F 2 "my_footprints:ADTS648_V" H 5700 3500 50  0001 C CNN
 F 3 "" H 5700 3500 50  0001 C CNN
-F 4 "Mouser" H 5700 3500 50  0001 C CNN "Supplier"
-F 5 "642-ADTS24NV" H 5700 3500 50  0001 C CNN "Supplier Order Code"
+F 4 "Mouser" H 5700 3500 50  0001 C CNN "Supplier 1"
+F 5 "642-ADTS648RV" H 5700 3500 50  0001 C CNN "Supplier 1 Order Code"
+F 6 "Digikey" H 5700 3500 50  0001 C CNN "Supplier 2"
+F 7 "679-2377-ND" H 5700 3500 50  0001 C CNN "Supplier 2 Order Code"
 	1    5700 3500
 	0    1    1    0
@@
 P 6500 4750
 F 0 "SW?" H 6600 4796 50  0000 L CNN
-F 1 "CAP_BROWN_6mm" H 6600 4705 50  0000 L CNN
+F 1 "CAP_GREEN_6mm" H 6600 4705 50  0000 L CNN
 F 2 "" H 6500 4750 50  0001 C CNN
 F 3 "~" H 6500 4750 50  0001 C CNN
-F 4 "Mouser" H 6500 4750 50  0001 C CNN "Supplier"
+F 4 "Mouser" H 6500 4750 50  0001 C CNN "Supplier 1"
+F 5 "642-AKTSC61G" H 6500 4750 50  0001 C CNN "Supplier 1 Order Code"
 	1    6500 4750
 	1    0    0    -1
@@
 F 0 "SW?" V 5654 4980 50  0000 L CNN
 F 1 "SW_6mm" V 5745 4980 50  0000 L CNN
-F 2 "" H 5700 4750 50  0001 C CNN
+F 2 "my_footprints:ADTS24_V" H 5700 4750 50  0001 C CNN
 F 3 "" H 5700 4750 50  0001 C CNN
-F 4 "Mouser" H 5700 4750 50  0001 C CNN "Supplier"
-F 5 "642-ADTS24NV" H 5700 4750 50  0001 C CNN "Supplier Order Code"
+F 4 "Mouser" H 5700 4750 50  0001 C CNN "Supplier 1"
+F 5 "642-ADTS24NV" H 5700 4750 50  0001 C CNN "Supplier 1 Order Code"
+F 6 "Digikey" H 5700 4750 50  0001 C CNN "Supplier 2"
+F 7 "679-2374-ND" H 5700 4750 50  0001 C CNN "Supplier 2 Order Code"
 	1    5700 4750
 	0    1    1    0
