File: PCB_rev0/binulator_kicad_project/file5B9A31FE.sch (KiCad schematic (older format))
At the start: 16 parts

Commit message: change power ICs to use a dedicated charge solution, add FTDI chip for serial comms over USB
Parts:
- removed Q?: MMBT3904, Package_TO_SOT_SMD:SOT-23, symbol Transistor_BJT:MMBT3904
- removed Q?: DMP3099L-7, Package_TO_SOT_SMD:SOT-23, symbol Device:Q_PMOS_GSD
- removed R? (x3): 1M2, symbol Device:R
- removed R?: 200k, symbol Device:R
- removed U?: BQ24040, my_footprints:S-PWSON-N10, symbol my_symbols:BQ2404x
- removed U?: TLV6703, Package_TO_SOT_SMD:SOT-23-6_Handsoldering, symbol my_symbols:TLV6703
- added C?: 10nF, symbol Device:C
- added C?: 0.1uF, symbol Device:C
- added R? (x2): 27R, symbol Device:R
- added U?: BQ24230, my_footprints:BQ24230, symbol my_symbols:BQ24230
- added U?: FT230XQ, Package_DFN_QFN:QFN-16-1EP_4x4mm_P0.65mm_EP2.5x2.5mm, symbol Interface_USB:FT230XQ
Connections:
- net labels added: FT230_RST, FT230_RXD, FT230_TXD, USB_D+, USB_D-, VBUS, ~FT230_CTS, ~FT230_RTS
- wire segments 66 -> 64
- no-connect marks 2 -> 1
Other:
- note added: "Battery - 18650 cell - https://www.jaycar.com.au/18650-2600mah-li-ion-protected-battery/p/SB2299"
- note removed: "Use a TLV6703 + pmos as a UVLO"
- note removed: "battery management IC\nbq2404x"

Commit message: add more to power schematic. VBUS sense divider, connect BQ24230 components, connect to VREG
Parts:
- removed C?: 10nF, symbol Device:C
- added 1k5, 47k+ (x2): R, symbol Device:R
- added 1k?: 1k5, symbol Device:R
- added C? (x2): 4.7uF, symbol Device:C
- added C?: 1uF, symbol Device:C
- added D? (x2): GRN LED - LTST-C281KGKT, symbol Device:LED
- added R?: 10k, symbol Device:R
- added R?: 3k60, symbol Device:R
- added R?: 1k8, symbol Device:R
Connections:
- net labels added: 3V3, VBUS_SENSE
- wire segments 64 -> 109
Other:
- note added: "Fast charge rate of (500mA ish)"
- note added: "Not using an NTC"
